Commit message: Camera views in RViz; thrust and fan air-flow effects in Gazebo and RViz
Gazebo: 12 particle emitters on the car (one per nozzle exit along its
exhaust, two fan exhausts on the rear deck), switched and rate-scaled by
the actuation system from the live (lagged) thrust and fan speed via
ignition.msgs.ParticleEmitter, published only on change. Soft round puff
texture (scripts/generate_puff_texture.py) instead of hard squares. The
emitters' +X is the emission axis (checked by screenshot).

Worlds: sensors system (ogre2) + particle-emitter2 system in every stunt
world; the ramp world gets a static trackside camera filming run-in, loop
and landing side-on (/camera/trackside, 640x400 @ 15 Hz).

RViz (demo_a.launch.py): image panels for the trackside camera and the
car's onboard camera (onboard_camera:=true by default), and
/stunt/viz_flow: exhaust puffs launched from every firing nozzle and the
fan vents in the world frame, growing and fading so they trail behind the
car through the flip, a fan disc glowing with fan speed, and animated
suction streaks converging into it.

Checked on a full Demo A run: frames captured from both cameras at the
inverted hold, drive-off, flip and landing burn show the plumes; RViz up,
mission reaches STOPPED.

File: src/roadster_description/urdf/roadster.urdf.xacro (robot description, xacro)
@@ -40,4 +40,6 @@
        against a ceiling hold from t = 0 instead of falling during spin-up) -->
     <xacro:arg name="surfaces_file" default="" />
+    <!-- cosmetic Gazebo particle plumes on the nozzles and fan exhausts -->
+    <xacro:arg name="with_effects" default="true" />
     <xacro:arg name="fan_initial_speed" default="0.0" />
     <!-- ===================== PHYSICAL PARAMETERS ===================== -->
@@ -436,6 +438,64 @@
                 <initial_speed>$(arg fan_initial_speed)</initial_speed>
             </fan>
+            <!-- drive the particle emitters below (rate = level x rate_max per s) -->
+            <effects>
+                <enabled>$(arg with_effects)</enabled>
+                <rate_max>200</rate_max>
+                <fan_rate_max>120</fan_rate_max>
+                <topic_prefix>/roadster/fx</topic_prefix>
+            </effects>
         </plugin>
     </gazebo>
+    <!-- ===================== VISUAL EFFECTS (Gazebo particles) ===================== -->
+    <!-- Cosmetic only, no physics. One emitter per nozzle at its exit, its +X
+       along the EXHAUST (opposite force_dir), so a firing nozzle shows a white
+       cold-gas plume; two on the rear deck show the suction fans' exhaust (the
+       ducted fans pull air from under the floor and blow it out above). All
+       start off; the actuation system switches them and sets their rate from
+       the live thrust / fan speed on /roadster/fx/<name>. Needs the world to
+       load ignition-gazebo-particle-emitter2-system. Attached to base_link
+       (the root link sdformat keeps) with explicit poses, so lumping cannot
+       move them. -->
+    <xacro:macro name="fx_emitter" params="name xyz exhaust rgb">
+        <particle_emitter name="fx_${name}" type="point">
+            <pose>${xyz[0]} ${xyz[1]} ${xyz[2] + wheel_radius} 0 ${-atan2(exhaust[2], sqrt(exhaust[0]*exhaust[0] + exhaust[1]*exhaust[1]))} ${atan2(exhaust[1], exhaust[0])}</pose>
+            <emitting>false</emitting>
+            <size>0.05 0.05 0.05</size>
+            <particle_size>0.4 0.4 0.4</particle_size>
+            <lifetime>0.5</lifetime>
+            <rate>0</rate>
+            <min_velocity>10</min_velocity>
+            <max_velocity>16</max_velocity>
+            <scale_rate>3</scale_rate>
+            <color_start>${rgb} 0.9</color_start>
+            <color_end>${rgb} 0.0</color_end>
+            <topic>/roadster/fx/${name}</topic>
+            <!-- soft round puff (scripts/generate_puff_texture.py) instead of hard squares -->
+            <material>
+                <diffuse>1 1 1 1</diffuse>
+                <pbr>
+                    <metal>
+                        <albedo_map>$(find roadster_description)/models/fx/puff.png</albedo_map>
+                    </metal>
+                </pbr>
+            </material>
+        </particle_emitter>
+    </xacro:macro>
+    <xacro:macro name="fx_nozzles" params="names">
+        <xacro:if value="${len(names) > 0}">
+            <xacro:fx_emitter name="${names[0]}" xyz="${nozzles[names[0]]['xyz']}"
+                exhaust="${[-c for c in nozzles[names[0]]['force_dir']]}" rgb="0.95 0.95 1.0" />
+            <xacro:fx_nozzles names="${names[1:]}" />
+        </xacro:if>
+    </xacro:macro>
+    <xacro:if value="$(arg with_effects)">
+        <gazebo reference="base_link">
+            <xacro:fx_nozzles names="${python.sorted(nozzles.keys())}" />
+            <xacro:fx_emitter name="fan_left" xyz="${[-1.8, 0.5, 0.7]}"
+                exhaust="${[-0.45, 0.0, 0.89]}" rgb="0.55 0.8 1.0" />
+            <xacro:fx_emitter name="fan_right" xyz="${[-1.8, -0.5, 0.7]}"
+                exhaust="${[-0.45, 0.0, 0.89]}" rgb="0.55 0.8 1.0" />
+        </gazebo>
+    </xacro:if>
     <!-- ===================== OPTIONAL RGB-D CAMERA ===================== -->
     <!-- verbatim from sedan.urdf.xacro (424x300, hfov 1.9, 10 Hz, far 50 m);

Commit message: Fly Demo A on the IMU estimate: 1 kHz IMU, suspension, no steering
IMU state estimate: the Gazebo IMU sampled instantaneous values at 200 Hz
while the rigid wheels took ~1 ms contact impulses (up to 150 m/s^2) at
every box-chain facet of the ramp; the aliased spikes drove the estimate
off by metres and up to 14 deg on the climb. The IMU now samples every
physics step (1 kHz, the simulated equivalent of a real IMU's
anti-alias filter) and the estimator integrates every sample, publishing
at 200 Hz on the sim-time grid. Estimate error over a whole Demo A: under
5 cm and 0.3 deg (flight phases under 1 cm). Found with ins_replay, an
offline replay of a recorded run through the exact filter.

Suspension: one preloaded spring-damper per corner (prismatic joints,
k = 250 kN/m, zeta 0.5, +-12 cm), applied by the actuation system as a
joint force (an SDF joint spring under this DART build did not deflect in
proportion to 1/k). The rigid car was statically indeterminate and rode on
one diagonal, halving the driven wheels on the climb; touchdown peak also
falls from 8-11 g to 5.6 g. Rest geometry unchanged (joints at 0 at 1 g).

Mission: steering off by default (straight track, no disturbance; small
estimate errors only twisted the car), fans spin up 6 m before the ramp,
the inverted hold stands still instead of chasing the estimate, speed is
read from the estimator's twist rather than differenced corrected poses,
inertia updated for the suspension links.

IMU-flown Demo A (state:=imu): hold 2.0 s still to 0.7 cm, all wheels
loaded run-in to drive-off (>= 1.5 kN), release 7.2 m/s, 180.0 deg flip,
touchdown 2.8 m/s / 0.07 deg / 5.6 g, rollout to a stop. Drop test still
passes. Zero-g force-point and ceiling-hold tests pass.

File: src/roadster_description/urdf/roadster.urdf.xacro (robot description, xacro)
@@ -26,10 +26,11 @@
        declared here. -->
     <xacro:arg name="with_camera" default="false" />
-    <!-- 1730 kg chassis + 4 x 15 kg wheels + 2 x 5 kg steer links = 1,800 kg total,
+    <!-- 1690 kg chassis + 4 x 10 kg suspension links + 4 x 15 kg wheels + 2 x 5 kg
+       steer links = 1,800 kg total (1730 before the suspension was added),
        the plan's nominal mass. The sedan stays at 300 kg "for stability"; this
        mass was verified stable on the 1 ms DART flat-runway smoke test
        (2026-10-16: wheel loads = sprung weight within 0.1%, traction-limited
        0-60 in 2.30 s at both 300 and 1,800 kg). -->
-    <xacro:arg name="chassis_mass" default="1730" />
+    <xacro:arg name="chassis_mass" default="1690" />
     <xacro:arg name="tire_mu" default="1.2" />
     <xacro:arg name="controllers_file"
@@ -145,10 +146,51 @@
         <xacro:box_inertia m="${ch_mass}" x="${ch_l}" y="${ch_w}" z="${ch_h + body_h}" />
     </link>
+    <!-- ===================== SUSPENSION MACRO ===================== -->
+    <!-- One vertical spring-damper per corner (prismatic, +z = the wheel moves
+       up relative to the chassis = compression). Without it the rigid car on
+       four rigid wheels is statically indeterminate: the physics engine can put
+       all the load on one diagonal, and did - traction control then had only two
+       driven wheels and the climb sagged from 6 to 2.4 m/s (IMU-flown run
+       imu_fly1, 2026-10-16); touchdown also peaked at 8-11 g.
+       Sized for stunt loads, not road loads: ~4-5 g at the ramp bottom (fan +
+       centripetal) means ~20 kN per corner, so k = 250 kN/m (~8 cm there) with
+       +-0.12 m travel, damping at zeta ~0.5 on a corner's sprung mass.
+       PRELOADED: at q = 0 each spring pushes with the quarter-chassis weight,
+       so at rest (1 g) the joints sit at 0, keeping base_link at ground level
+       and the chassis frame wheel_radius above it - constants the mission,
+       estimator, analyzer and tests rely on.
+       The spring-damper force is applied by the actuation system (JointForceCmd
+       every physics step, <suspension> in its plugin block below): an SDF joint
+       spring in this Fortress / DART build gave static deflections that did not
+       scale with k (the implied corner load went from 5.9 to 6.5 kN between
+       k = 250 and 500 kN/m), so it could not be trusted. -->
+    <xacro:property name="susp_k" value="250000.0" />
+    <xacro:property name="susp_travel" value="0.12" />
+    <xacro:property name="susp_mass" value="10.0" />
+    <!-- each spring carries a quarter of the chassis (steer links and wheels hang below it) -->
+    <xacro:property name="susp_preload" value="${ch_mass * 9.81 / 4.0}" />
+    <xacro:property name="susp_damping" value="${2.0 * 0.5 * sqrt(susp_k * ch_mass / 4.0)}" />
+    <xacro:macro name="suspension" params="prefix x_off y_off">
+        <joint name="${prefix}_suspension_joint" type="prismatic">
+            <parent link="chassis" />
+            <child link="${prefix}_suspension_link" />
+            <origin xyz="${x_off} ${y_off} 0" rpy="0 0 0" />
+            <axis xyz="0 0 1" />
+            <limit lower="${-susp_travel}" upper="${susp_travel}" effort="100000.0" velocity="10.0" />
+            <dynamics damping="0.0" />
+        </joint>
+        <link name="${prefix}_suspension_link">
+            <inertial>
+                <mass value="${susp_mass}" />
+                <inertia ixx="0.05" ixy="0" ixz="0" iyy="0.05" iyz="0" izz="0.05" />
+            </inertial>
+        </link>
+    </xacro:macro>
     <!-- ===================== STEERING LINK MACRO ===================== -->
     <xacro:macro name="steering_link" params="prefix x_off y_off">
         <joint name="${prefix}_wheel_steering_joint" type="revolute">
-            <parent link="chassis" />
+            <parent link="${prefix}_suspension_link" />
             <child link="${prefix}_wheel_steering_link" />
-            <origin xyz="${x_off} ${y_off} 0" rpy="0 0 0" />
+            <origin xyz="0 0 0" rpy="0 0 0" />
             <axis xyz="0 0 1" />
             <!-- same mechanical stop and rate as the sedan; the drive
@@ -209,4 +251,8 @@
     </xacro:macro>
     <!-- ===================== INSTANTIATE ===================== -->
+    <xacro:suspension prefix="front_left" x_off="${wheelbase/2}" y_off="${track_width/2}" />
+    <xacro:suspension prefix="front_right" x_off="${wheelbase/2}" y_off="${-track_width/2}" />
+    <xacro:suspension prefix="rear_left" x_off="${-wheelbase/2}" y_off="${track_width/2}" />
+    <xacro:suspension prefix="rear_right" x_off="${-wheelbase/2}" y_off="${-track_width/2}" />
     <xacro:steering_link prefix="front_left" x_off="${wheelbase/2}" y_off="${track_width/2}" />
     <xacro:steering_link prefix="front_right" x_off="${wheelbase/2}" y_off="${-track_width/2}" />
@@ -216,7 +262,7 @@
         parent="front_right_wheel_steering_link" x_off="0" y_off="0" z_off="0" />
     <xacro:wheel name="rear_left_wheel"
-        parent="chassis" x_off="${-wheelbase/2}" y_off="${track_width/2}" z_off="0" />
+        parent="rear_left_suspension_link" x_off="0" y_off="0" z_off="0" />
     <xacro:wheel name="rear_right_wheel"
-        parent="chassis" x_off="${-wheelbase/2}" y_off="${-track_width/2}" z_off="0" />
+        parent="rear_right_suspension_link" x_off="0" y_off="0" z_off="0" />
     <!-- ===================== WHEEL FRICTION ===================== -->
     <!-- same <gazebo reference><collision> blob path as the sedan (slip1/slip2
@@ -326,9 +372,14 @@
         </xacro:element>
     </xacro:macro>
-    <!-- same noise model as the sedan. 200 Hz (sedan: 100) for the attitude loop. -->
+    <!-- same noise model as the sedan. 1 kHz = the physics step (sedan: 100 Hz):
+       the rigid wheels on the box-chain ramp take ~1 ms contact impulses (up to
+       150 m/s^2) at every facet joint; sampled at 200 Hz an instantaneous IMU
+       aliases them (a 1 ms spike integrated over 5 ms), which drove the IMU
+       state estimate off by metres on the climb. A real IMU low-pass filters
+       before sampling; sampling every physics step is the simulated equivalent. -->
     <gazebo reference="imu_link">
         <sensor name="imu_sensor" type="imu">
             <always_on>true</always_on>
-            <update_rate>200</update_rate>
+            <update_rate>1000</update_rate>
             <topic>imu</topic>
             <ignition_frame_id>imu_link</ignition_frame_id>
@@ -391,4 +442,17 @@
         <xacro:position_steer joint="front_left_wheel_steering_joint" />
         <xacro:position_steer joint="front_right_wheel_steering_joint" />
+        <!-- suspension: passive springs, state only (joint_state_broadcaster
+           publishes them so robot_state_publisher can place the wheels, and the
+           state estimator reads the travel for its wheel-centre lever) -->
+        <xacro:macro name="passive_joint" params="joint">
+            <joint name="${joint}">
+                <state_interface name="position" />
+                <state_interface name="velocity" />
+            </joint>
+        </xacro:macro>
+        <xacro:passive_joint joint="front_left_suspension_joint" />
+        <xacro:passive_joint joint="front_right_suspension_joint" />
+        <xacro:passive_joint joint="rear_left_suspension_joint" />
+        <xacro:passive_joint joint="rear_right_suspension_joint" />
     </ros2_control>
     <gazebo>
@@ -438,4 +502,13 @@
                 <initial_speed>$(arg fan_initial_speed)</initial_speed>
             </fan>
+            <!-- suspension spring-dampers (see the SUSPENSION MACRO comment):
+               joint force = -(preload + k q + c dq/dt) -->
+            <suspension>
+                <joints>front_left_suspension_joint front_right_suspension_joint
+                    rear_left_suspension_joint rear_right_suspension_joint</joints>
+                <stiffness>${susp_k}</stiffness>
+                <damping>${susp_damping}</damping>
+                <preload>${susp_preload}</preload>
+            </suspension>
             <!-- drive the particle emitters below (rate = level x rate_max per s) -->
             <effects>

Commit message: air jets adjustment

File: src/roadster_description/urdf/roadster.urdf.xacro (robot description, xacro)
@@ -515,8 +515,10 @@
                 <preload>${susp_preload}</preload>
             </suspension>
-            <!-- drive the particle emitters below (rate = level x rate_max per s) -->
+            <!-- drive the particle emitters below (rate = level x rate_max per s,
+               at least 0.1 x rate_max): the nozzle jets need a high rate so
+               even a partial-thrust jet stays one continuous column -->
             <effects>
                 <enabled>$(arg with_effects)</enabled>
-                <rate_max>200</rate_max>
+                <rate_max>2000</rate_max>
                 <fan_rate_max>120</fan_rate_max>
                 <topic_prefix>/roadster/fx</topic_prefix>
@@ -533,25 +535,34 @@
        load ignition-gazebo-particle-emitter2-system. Attached to base_link
        (the root link sdformat keeps) with explicit poses, so lumping cannot
-       move them. -->
-    <xacro:macro name="fx_emitter" params="name xyz exhaust rgb">
+       move them.
+       Nozzle jets (style jet), after the photographed cold-gas jets
+       (docs/snapshots/tesla_roadster2_thrusters.jpg): a narrow, dense column.
+       Small, fast particles at a high rate overlap heavily; the faint Gaussian
+       texture (jet.png) makes the overlap a bright core with soft edges (a
+       dense texture saturates into a hard white rod), and a narrow speed
+       spread keeps the column smooth (a wide one clumps it into beads).
+       Fan exhaust (style puff): sparse soft puffs (puff.png) that grow into a
+       haze. -->
+    <xacro:macro name="fx_emitter" params="name xyz exhaust rgb style">
+        <xacro:property name="jet" value="${style == 'jet'}" />
         <particle_emitter name="fx_${name}" type="point">
             <pose>${xyz[0]} ${xyz[1]} ${xyz[2] + wheel_radius} 0 ${-atan2(exhaust[2], sqrt(exhaust[0]*exhaust[0] + exhaust[1]*exhaust[1]))} ${atan2(exhaust[1], exhaust[0])}</pose>
             <emitting>false</emitting>
             <size>0.05 0.05 0.05</size>
-            <particle_size>0.4 0.4 0.4</particle_size>
-            <lifetime>0.5</lifetime>
+            <particle_size>${'0.18 0.18 0.18' if jet else '0.4 0.4 0.4'}</particle_size>
+            <lifetime>${0.15 if jet else 0.5}</lifetime>
             <rate>0</rate>
-            <min_velocity>10</min_velocity>
-            <max_velocity>16</max_velocity>
-            <scale_rate>3</scale_rate>
+            <min_velocity>${19 if jet else 10}</min_velocity>
+            <max_velocity>${21 if jet else 16}</max_velocity>
+            <scale_rate>${2 if jet else 3}</scale_rate>
             <color_start>${rgb} 0.9</color_start>
             <color_end>${rgb} 0.0</color_end>
             <topic>/roadster/fx/${name}</topic>
-            <!-- soft round puff (scripts/generate_puff_texture.py) instead of hard squares -->
+            <!-- soft round textures from scripts/generate_puff_texture.py instead of hard squares -->
             <material>
                 <diffuse>1 1 1 1</diffuse>
                 <pbr>
                     <metal>
-                        <albedo_map>$(find roadster_description)/models/fx/puff.png</albedo_map>
+                        <albedo_map>$(find roadster_description)/models/fx/${style}.png</albedo_map>
                     </metal>
                 </pbr>
@@ -562,5 +573,6 @@
         <xacro:if value="${len(names) > 0}">
             <xacro:fx_emitter name="${names[0]}" xyz="${nozzles[names[0]]['xyz']}"
-                exhaust="${[-c for c in nozzles[names[0]]['force_dir']]}" rgb="0.95 0.95 1.0" />
+                exhaust="${[-c for c in nozzles[names[0]]['force_dir']]}" rgb="0.95 0.95 1.0"
+                style="jet" />
             <xacro:fx_nozzles names="${names[1:]}" />
         </xacro:if>
@@ -570,7 +582,7 @@
             <xacro:fx_nozzles names="${python.sorted(nozzles.keys())}" />
             <xacro:fx_emitter name="fan_left" xyz="${[-1.8, 0.5, 0.7]}"
-                exhaust="${[-0.45, 0.0, 0.89]}" rgb="0.55 0.8 1.0" />
+                exhaust="${[-0.45, 0.0, 0.89]}" rgb="0.55 0.8 1.0" style="puff" />
             <xacro:fx_emitter name="fan_right" xyz="${[-1.8, -0.5, 0.7]}"
-                exhaust="${[-0.45, 0.0, 0.89]}" rgb="0.55 0.8 1.0" />
+                exhaust="${[-0.45, 0.0, 0.89]}" rgb="0.55 0.8 1.0" style="puff" />
         </gazebo>
     </xacro:if>
